Commit message: updated urdf

File: vacu_bot/urdf/vacu_bot.urdf.xacro (robot description, xacro)
@@ -62,14 +62,14 @@
           rgba="0.8 0.8 0.8 1" />
       </material>
-      <origin rpy="1.57075 0 1.57075" xyz="0 0 0"/>
-    </visual>
-    <collision>
-      <geometry>
-        <cylinder length="0.1" radius="0.05"/>
-      </geometry>
-      <origin rpy="1.57075 0 1.57075" xyz="0 0 0"/>
-    </collision>
-    <xacro:cylinder_inertial radius="0.05" length="0.1" mass="1">
-        <origin xyz="0.0 0.2 0.0" rpy="0 0 0"/>
+      <origin rpy="1.57075 0 0" xyz="0 0 0"/>
+    </visual>
+    <collision>
+      <geometry>
+        <cylinder length="0.1" radius="0.05"/>
+      </geometry>
+      <origin rpy="1.57075 0 0" xyz="0 0 0"/>
+    </collision>
+    <xacro:cylinder_inertial radius="0.05" length="0.1" mass="1">
+        <origin xyz="0.0 0.0 0.0" rpy="0 0 0"/>
     </xacro:cylinder_inertial>
   </link>
@@ -84,14 +84,14 @@
           rgba="0.8 0.8 0.8 1" />
       </material>
-      <origin rpy="1.57075 0 1.57075" xyz="0 0 0"/>
-    </visual>
-    <collision>
-      <geometry>
-        <cylinder length="0.1" radius="0.05"/>
-      </geometry>
-      <origin rpy="1.57075 0 1.57075" xyz="0 0 0"/>
-    </collision>
-    <xacro:cylinder_inertial radius="0.05" length="0.1" mass="1">
-        <origin xyz="0.0 0.2 0.0" rpy="0 0 0"/>
+      <origin rpy="1.57075 0 0" xyz="0 0 0"/>
+    </visual>
+    <collision>
+      <geometry>
+        <cylinder length="0.1" radius="0.05"/>
+      </geometry>
+      <origin rpy="1.57075 0 0" xyz="0 0 0"/>
+    </collision>
+    <xacro:cylinder_inertial radius="0.05" length="0.1" mass="1">
+        <origin xyz="0.0 0.0 0.0" rpy="0 0 0"/>
     </xacro:cylinder_inertial>
   </link>
@@ -106,14 +106,14 @@
           rgba="0.8 0.8 0.8 1" />
       </material>
-      <origin rpy="1.57075 0 1.57075" xyz="0 0 0"/>
-    </visual>
-    <collision>
-      <geometry>
-        <cylinder length="0.1" radius="0.05"/>
-      </geometry>
-      <origin rpy="1.57075 0 1.57075" xyz="0 0 0"/>
-    </collision>
-    <xacro:cylinder_inertial radius="0.05" length="0.1" mass="1">
-        <origin xyz="0.2 -0.2 0.0" rpy="0 0 0"/>
+      <origin rpy="1.57075 0 0" xyz="0 0 0"/>
+    </visual>
+    <collision>
+      <geometry>
+        <cylinder length="0.1" radius="0.05"/>
+      </geometry>
+      <origin rpy="1.57075 0 0" xyz="0 0 0"/>
+    </collision>
+    <xacro:cylinder_inertial radius="0.05" length="0.1" mass="1">
+        <origin xyz="0.0 0.0 0.0" rpy="0 0 0"/>
     </xacro:cylinder_inertial>
   </link>
@@ -128,14 +128,14 @@
           rgba="0.8 0.8 0.8 1" />
       </material>
-      <origin rpy="1.57075 0 1.57075" xyz="0 0 0"/>
-    </visual>
-    <collision>
-      <geometry>
-        <cylinder length="0.1" radius="0.05"/>
-      </geometry>
-      <origin rpy="1.57075 0 1.57075" xyz="0 0 0"/>
-    </collision>
-    <xacro:cylinder_inertial radius="0.05" length="0.1" mass="1">
-        <origin xyz="-0.2 -0.2 0.0" rpy="0 0 0"/>
+      <origin rpy="1.57075 0 0" xyz="0 0 0"/>
+    </visual>
+    <collision>
+      <geometry>
+        <cylinder length="0.1" radius="0.05"/>
+      </geometry>
+      <origin rpy="1.57075 0 0" xyz="0 0 0"/>
+    </collision>
+    <xacro:cylinder_inertial radius="0.05" length="0.1" mass="1">
+        <origin xyz="0.0 0.0 0.0" rpy="0 0 0"/>
     </xacro:cylinder_inertial>
   </link>
@@ -157,8 +157,8 @@
          <cylinder length="0.2" radius="0.05"/>
       </geometry>
-      <origin rpy="0 0 0.4" xyz="0 0 0"/>
+      <origin rpy="0 0 0" xyz="0 0 0"/>
     </collision>
     <xacro:cylinder_inertial radius="0.05" length="0.1" mass="0.5">
-        <origin xyz="0.0 0.0 0.2" rpy="0 0 0"/>
+        <origin xyz="0.0 0.0 0.0" rpy="0 0 0"/>
     </xacro:cylinder_inertial>
   </link>
@@ -173,9 +173,11 @@
     <child link="front_left_wheel"/>
     <origin xyz="0.35 -0.275 -0.15"/>
+    <axis xyz="0 1 0"/>
   </joint>
   <joint name="base_to_front_right_wheel" type="continuous">
     <parent link="base_link"/>
     <child link="front_right_wheel"/>
-    <origin xyz="-0.35 -0.275 -0.15"/>
+    <origin xyz="0.35 0.275 -0.15"/>
+    <axis xyz="0 1 0"/>
   </joint>
   <joint name="base_to_rear_right_wheel" type="continuous">
@@ -183,9 +185,11 @@
     <child link="rear_right_wheel"/>
     <origin xyz="-0.35 0.275 -0.15"/>
+    <axis xyz="0 1 0"/>
   </joint>
   <joint name="base_to_rear_left_wheel" type="continuous">
     <parent link="base_link"/>
     <child link="rear_left_wheel"/>
-    <origin xyz="0.35 0.275 -0.15"/>
+    <origin xyz="-0.35 -0.275 -0.15"/>
+    <axis xyz="0 1 0"/>
   </joint>
   <joint name="base_to_lidar" type="fixed">

Commit message: changes in urdf and launch and rviz

File: vacu_bot/urdf/vacu_bot.urdf.xacro (robot description, xacro)
@@ -62,11 +62,11 @@
           rgba="0.8 0.8 0.8 1" />
       </material>
-      <origin rpy="1.57075 0 1.57075" xyz="0 0 0"/>
-    </visual>
-    <collision>
-      <geometry>
-        <cylinder length="0.1" radius="0.05"/>
-      </geometry>
-      <origin rpy="1.57075 0 1.57075" xyz="0 0 0"/>
+      <origin rpy="1.57075 0 0" xyz="0 0 0"/>
+    </visual>
+    <collision>
+      <geometry>
+        <cylinder length="0.1" radius="0.05"/>
+      </geometry>
+      <origin rpy="1.57075 0 0" xyz="0 0 0"/>
     </collision>
     <xacro:cylinder_inertial radius="0.05" length="0.1" mass="1">
@@ -84,11 +84,11 @@
           rgba="0.8 0.8 0.8 1" />
       </material>
-      <origin rpy="1.57075 0 1.57075" xyz="0 0 0"/>
-    </visual>
-    <collision>
-      <geometry>
-        <cylinder length="0.1" radius="0.05"/>
-      </geometry>
-      <origin rpy="1.57075 0 1.57075" xyz="0 0 0"/>
+      <origin rpy="1.57075 0 0" xyz="0 0 0"/>
+    </visual>
+    <collision>
+      <geometry>
+        <cylinder length="0.1" radius="0.05"/>
+      </geometry>
+      <origin rpy="1.57075 0 0" xyz="0 0 0"/>
     </collision>
     <xacro:cylinder_inertial radius="0.05" length="0.1" mass="1">
@@ -106,11 +106,11 @@
           rgba="0.8 0.8 0.8 1" />
       </material>
-      <origin rpy="1.57075 0 1.57075" xyz="0 0 0"/>
-    </visual>
-    <collision>
-      <geometry>
-        <cylinder length="0.1" radius="0.05"/>
-      </geometry>
-      <origin rpy="1.57075 0 1.57075" xyz="0 0 0"/>
+      <origin rpy="1.57075 0 0" xyz="0 0 0"/>
+    </visual>
+    <collision>
+      <geometry>
+        <cylinder length="0.1" radius="0.05"/>
+      </geometry>
+      <origin rpy="1.57075 0 0" xyz="0 0 0"/>
     </collision>
     <xacro:cylinder_inertial radius="0.05" length="0.1" mass="1">
@@ -128,11 +128,11 @@
           rgba="0.8 0.8 0.8 1" />
       </material>
-      <origin rpy="1.57075 0 1.57075" xyz="0 0 0"/>
-    </visual>
-    <collision>
-      <geometry>
-        <cylinder length="0.1" radius="0.05"/>
-      </geometry>
-      <origin rpy="1.57075 0 1.57075" xyz="0 0 0"/>
+      <origin rpy="1.57075 0 0" xyz="0 0 0"/>
+    </visual>
+    <collision>
+      <geometry>
+        <cylinder length="0.1" radius="0.05"/>
+      </geometry>
+      <origin rpy="1.57075 0 0" xyz="0 0 0"/>
     </collision>
     <xacro:cylinder_inertial radius="0.05" length="0.1" mass="1">
@@ -172,20 +172,24 @@
     <parent link="base_link"/>
     <child link="front_left_wheel"/>
+    <origin xyz="0.35 0.275 -0.15"/>
+    <axis xyz="0 1 0"/>
+  </joint>
+  <joint name="base_to_front_right_wheel" type="continuous">
+    <parent link="base_link"/>
+    <child link="front_right_wheel"/>
     <origin xyz="0.35 -0.275 -0.15"/>
-  </joint>
-  <joint name="base_to_front_right_wheel" type="continuous">
-    <parent link="base_link"/>
-    <child link="front_right_wheel"/>
+    <axis xyz="0 1 0"/>
+  </joint>
+  <joint name="base_to_rear_right_wheel" type="continuous">
+    <parent link="base_link"/>
+    <child link="rear_right_wheel"/>
     <origin xyz="-0.35 -0.275 -0.15"/>
-  </joint>
-  <joint name="base_to_rear_right_wheel" type="continuous">
-    <parent link="base_link"/>
-    <child link="rear_right_wheel"/>
+    <axis xyz="0 1 0"/>
+  </joint>
+  <joint name="base_to_rear_left_wheel" type="continuous">
+    <parent link="base_link"/>
+    <child link="rear_left_wheel"/>
     <origin xyz="-0.35 0.275 -0.15"/>
-  </joint>
-  <joint name="base_to_rear_left_wheel" type="continuous">
-    <parent link="base_link"/>
-    <child link="rear_left_wheel"/>
-    <origin xyz="0.35 0.275 -0.15"/>
+    <axis xyz="0 1 0"/>
   </joint>
   <joint name="base_to_lidar" type="fixed">

Commit message: changes in urdf

File: vacu_bot/urdf/vacu_bot.urdf.xacro (robot description, xacro)
@@ -71,5 +71,5 @@
     </collision>
     <xacro:cylinder_inertial radius="0.05" length="0.1" mass="1">
-        <origin xyz="0.0 0.2 0.0" rpy="0 0 0"/>
+        <origin xyz="0.0 0.0 0.0" rpy="0 0 0"/>
     </xacro:cylinder_inertial>
   </link>
@@ -93,5 +93,5 @@
     </collision>
     <xacro:cylinder_inertial radius="0.05" length="0.1" mass="1">
-        <origin xyz="0.0 0.2 0.0" rpy="0 0 0"/>
+        <origin xyz="0.0 0.0 0.0" rpy="0 0 0"/>
     </xacro:cylinder_inertial>
   </link>
@@ -115,5 +115,5 @@
     </collision>
     <xacro:cylinder_inertial radius="0.05" length="0.1" mass="1">
-        <origin xyz="0.2 -0.2 0.0" rpy="0 0 0"/>
+        <origin xyz="0.0 0.0 0.0" rpy="0 0 0"/>
     </xacro:cylinder_inertial>
   </link>
@@ -137,5 +137,5 @@
     </collision>
     <xacro:cylinder_inertial radius="0.05" length="0.1" mass="1">
-        <origin xyz="-0.2 -0.2 0.0" rpy="0 0 0"/>
+        <origin xyz="0.0 0.0 0.0" rpy="0 0 0"/>
     </xacro:cylinder_inertial>
   </link>
@@ -157,8 +157,8 @@
          <cylinder length="0.2" radius="0.05"/>
       </geometry>
-      <origin rpy="0 0 0.4" xyz="0 0 0"/>
+      <origin rpy="0 0 0.0" xyz="0 0 0"/>
     </collision>
     <xacro:cylinder_inertial radius="0.05" length="0.1" mass="0.5">
-        <origin xyz="0.0 0.0 0.2" rpy="0 0 0"/>
+        <origin xyz="0.0 0.0 0.0" rpy="0 0 0"/>
     </xacro:cylinder_inertial>
   </link>

Commit message: changes in urdf

File: vacu_bot/urdf/vacu_bot.urdf.xacro (robot description, xacro)
@@ -172,23 +172,23 @@
     <parent link="base_link"/>
     <child link="front_left_wheel"/>
+    <origin xyz="0.35 -0.275 -0.15"/>
+    <axis xyz="0 1 0"/>
+  </joint>
+  <joint name="base_to_front_right_wheel" type="continuous">
+    <parent link="base_link"/>
+    <child link="front_right_wheel"/>
     <origin xyz="0.35 0.275 -0.15"/>
     <axis xyz="0 1 0"/>
   </joint>
-  <joint name="base_to_front_right_wheel" type="continuous">
-    <parent link="base_link"/>
-    <child link="front_right_wheel"/>
-    <origin xyz="0.35 -0.275 -0.15"/>
-    <axis xyz="0 1 0"/>
-  </joint>
   <joint name="base_to_rear_right_wheel" type="continuous">
     <parent link="base_link"/>
     <child link="rear_right_wheel"/>
+    <origin xyz="-0.35 0.275 -0.15"/>
+    <axis xyz="0 1 0"/>
+  </joint>
+  <joint name="base_to_rear_left_wheel" type="continuous">
+    <parent link="base_link"/>
+    <child link="rear_left_wheel"/>
     <origin xyz="-0.35 -0.275 -0.15"/>
-    <axis xyz="0 1 0"/>
-  </joint>
-  <joint name="base_to_rear_left_wheel" type="continuous">
-    <parent link="base_link"/>
-    <child link="rear_left_wheel"/>
-    <origin xyz="-0.35 0.275 -0.15"/>
     <axis xyz="0 1 0"/>
   </joint>
