Commit message: delete fun_bot

File: vacu_bot/urdf/simu_gazebo_config.xacro (robot description, xacro)
@@ -30,6 +30,6 @@
      <updateRate>100.0</updateRate>
      <robotNamespace>/</robotNamespace>
-     <leftFrontJoint>base_to_left_front_wheel</leftFrontJoint>
-     <rightFrontJoint>base_to_right_front_wheel</rightFrontJoint>
+     <leftFrontJoint>base_to_front_left_wheel</leftFrontJoint>
+     <rightFrontJoint>base_to_front_right_wheel</rightFrontJoint>
      <leftRearJoint>base_to_rear_left_wheel</leftRearJoint>
      <rightRearJoint>base_to_rear_right_wheel</rightRearJoint>
@@ -46,4 +46,46 @@
   </gazebo>
  </xacro:macro>
+<!--############################## camera ################################################-->
+  <xacro:macro name="gazebo_camera" params="">
+   <gazebo reference="camera_link">
+     <sensor type="camera" name="camera1">
+       <update_rate>30.0</update_rate>
+       <camera name="head">
+         <horizontal_fov>1.3962634</horizontal_fov>
+         <image>
+           <width>800</width>
+           <height>800</height>
+           <format>R8G8B8</format>
+         </image>
+         <clip>
+           <near>0.02</near>
+           <far>300</far>
+         </clip>
+         <noise>
+           <type>gaussian</type>
+           <!-- Noise is sampled independently per pixel on each frame.
+                That pixel's noise value is added to each of its color
+                channels, which at that point lie in the range [0,1]. -->
+           <mean>0.0</mean>
+           <stddev>0.007</stddev>
+         </noise>
+      </camera>
+      <plugin name="camera_controller" filename="libgazebo_ros_camera.so">
+         <alwaysOn>true</alwaysOn>
+         <updateRate>0.0</updateRate>
+         <cameraName>vacu_bot/camera1</cameraName>
+         <imageTopicName>image_raw</imageTopicName>
+         <cameraInfoTopicName>camera_info</cameraInfoTopicName>
+         <frameName>camera_link</frameName>
+         <hackBaseline>0.07</hackBaseline>
+         <distortionK1>0.0</distortionK1>
+         <distortionK2>0.0</distortionK2>
+         <distortionK3>0.0</distortionK3>
+         <distortionT1>0.0</distortionT1>
+         <distortionT2>0.0</distortionT2>
+       </plugin>
+     </sensor>
+   </gazebo>
+  </xacro:macro>
 <!--############################## lidar ################################################-->
   <xacro:macro name="gazebo_lidar" params="">

File: vacu_bot/urdf/vacu_bot.urdf.xacro (robot description, xacro)
@@ -33,5 +33,5 @@
     <visual>
       <geometry>
-        <cylinder length="0.3" radius="0.5"/>
+        <cylinder length="0.4" radius="0.5"/>
       </geometry>
       <material
@@ -48,27 +48,5 @@
       <origin rpy="0 0 0" xyz="0 0 0"/>
     </collision>
-    <xacro:cylinder_inertial radius="0.5" length="0.3" mass="30">
-        <origin xyz="0.0 0.0 0.0" rpy="0 0 0"/>
-    </xacro:cylinder_inertial>
-  </link>
-  <link name="front_left_wheel">
-    <visual>
-      <geometry>
-        <cylinder length="0.1" radius="0.05"/>
-      </geometry>
-      <material
-        name="">
-        <color
-          rgba="0.8 0.8 0.8 1" />
-      </material>
-      <origin rpy="1.57075 0 0" xyz="0 0 0"/>
-    </visual>
-    <collision>
-      <geometry>
-        <cylinder length="0.1" radius="0.05"/>
-      </geometry>
-      <origin rpy="1.57075 0 0" xyz="0 0 0"/>
-    </collision>
-    <xacro:cylinder_inertial radius="0.05" length="0.1" mass="1">
+    <xacro:cylinder_inertial radius="0.5" length="0.4" mass="30">
         <origin xyz="0.0 0.0 0.0" rpy="0 0 0"/>
     </xacro:cylinder_inertial>
@@ -96,68 +74,114 @@
     </xacro:cylinder_inertial>
   </link>
-  <link name="rear_right_wheel">
-    <visual>
-      <geometry>
-        <cylinder length="0.1" radius="0.05"/>
-      </geometry>
-      <material
-        name="">
-        <color
-          rgba="0.8 0.8 0.8 1" />
-      </material>
-      <origin rpy="1.57075 0 0" xyz="0 0 0"/>
-    </visual>
-    <collision>
-      <geometry>
-        <cylinder length="0.1" radius="0.05"/>
-      </geometry>
-      <origin rpy="1.57075 0 0" xyz="0 0 0"/>
-    </collision>
-    <xacro:cylinder_inertial radius="0.05" length="0.1" mass="1">
-        <origin xyz="0.0 0.0 0.0" rpy="0 0 0"/>
-    </xacro:cylinder_inertial>
-  </link>
-  <link name="rear_left_wheel">
-    <visual>
-      <geometry>
-        <cylinder length="0.1" radius="0.05"/>
-      </geometry>
-      <material
-        name="">
-        <color
-          rgba="0.8 0.8 0.8 1" />
-      </material>
-      <origin rpy="1.57075 0 0" xyz="0 0 0"/>
-    </visual>
-    <collision>
-      <geometry>
-        <cylinder length="0.1" radius="0.05"/>
-      </geometry>
-      <origin rpy="1.57075 0 0" xyz="0 0 0"/>
-    </collision>
-    <xacro:cylinder_inertial radius="0.05" length="0.1" mass="1">
-        <origin xyz="0.0 0.0 0.0" rpy="0 0 0"/>
-    </xacro:cylinder_inertial>
-  </link>
+<!--############## selber gemacht #######-->
+   <link name="front_left_wheel">
+    <visual>
+      <geometry>
+        <cylinder length="0.1" radius="0.05"/>
+      </geometry>
+      <material
+        name="">
+        <color
+          rgba="0.8 0.8 0.8 1" />
+      </material>
+      <origin rpy="1.57075 0 0" xyz="0 0 0"/>
+    </visual>
+    <collision>
+      <geometry>
+        <cylinder length="0.1" radius="0.05"/>
+      </geometry>
+      <origin rpy="1.57075 0 0" xyz="0 0 0"/>
+    </collision>
+    <xacro:cylinder_inertial radius="0.05" length="0.1" mass="1">
+        <origin xyz="0.0 0.0 0.0" rpy="0 0 0"/>
+    </xacro:cylinder_inertial>
+  </link>
+   <link name="rear_right_wheel">
+    <visual>
+      <geometry>
+        <cylinder length="0.1" radius="0.05"/>
+      </geometry>
+      <material
+        name="">
+        <color
+          rgba="0.8 0.8 0.8 1" />
+      </material>
+      <origin rpy="1.57075 0 0" xyz="0 0 0"/>
+    </visual>
+    <collision>
+      <geometry>
+        <cylinder length="0.1" radius="0.05"/>
+      </geometry>
+      <origin rpy="1.57075 0 0" xyz="0 0 0"/>
+    </collision>
+    <xacro:cylinder_inertial radius="0.05" length="0.1" mass="1">
+        <origin xyz="0.0 0.0 0.0" rpy="0 0 0"/>
+    </xacro:cylinder_inertial>
+  </link>
+   <link name="rear_left_wheel">
+    <visual>
+      <geometry>
+        <cylinder length="0.1" radius="0.05"/>
+      </geometry>
+      <material
+        name="">
+        <color
+          rgba="0.8 0.8 0.8 1" />
+      </material>
+      <origin rpy="1.57075 0 0" xyz="0 0 0"/>
+    </visual>
+    <collision>
+      <geometry>
+        <cylinder length="0.1" radius="0.05"/>
+      </geometry>
+      <origin rpy="1.57075 0 0" xyz="0 0 0"/>
+    </collision>
+    <xacro:cylinder_inertial radius="0.05" length="0.1" mass="1">
+        <origin xyz="0.0 0.0 0.0" rpy="0 0 0"/>
+    </xacro:cylinder_inertial>
+  </link>
+ <!--#################################-->
 <!--############################################ sensor defintions ###################################-->
+   <link name="camera_link">
+    <visual>
+      <geometry>
+         <box size="0.1 0.1 0.1"/>
+      </geometry>
+      <material
+        name="">
+        <color
+          rgba="0.5 0.5 0.5 1" />
+      </material>
+      <origin rpy="0 0 0" xyz="0 0 0"/>
+    </visual>
+    <collision>
+      <geometry>
+         <box size="0.1 0.1 0.1"/>
+      </geometry>
+      <origin rpy="0 0 0" xyz="0 0 0"/>
+    </collision>
+    <xacro:box_inertial x="0.1" y="0.1" z="0.1" mass="0.5">
+        <origin xyz="0.0 0.0 0.0" rpy="0 0 0"/>
+    </xacro:box_inertial>
+  </link>
    <link name="lidar">
     <visual>
       <geometry>
-         <cylinder length="0.05" radius="0.1"/>
-      </geometry>
-      <material
-        name="">
-        <color
-          rgba="0.7 0 0 1" />
-      </material>
-      <origin rpy="0 0 0" xyz="0 0 0"/>
-    </visual>
-    <collision>
-      <geometry>
          <cylinder length="0.2" radius="0.05"/>
       </geometry>
-      <origin rpy="0 0 0.0" xyz="0 0 0"/>
-    </collision>
-    <xacro:cylinder_inertial radius="0.05" length="0.1" mass="0.5">
+      <material
+        name="">
+        <color
+          rgba="0.9 0.9 0.9 1" />
+      </material>
+      <origin rpy="0 0 0" xyz="0 0 0"/>
+    </visual>
+    <collision>
+      <geometry>
+         <cylinder length="0.2" radius="0.05"/>
+      </geometry>
+      <origin rpy="0 0 0" xyz="0 0 0"/>
+    </collision>
+    <xacro:cylinder_inertial radius="0.05" length="0.2" mass="0.5">
         <origin xyz="0.0 0.0 0.0" rpy="0 0 0"/>
     </xacro:cylinder_inertial>
@@ -167,34 +191,41 @@
     <parent link="base_footprint"/>
     <child link="base_link"/>
-    <origin xyz="0 0 0.15"/>
+    <origin xyz="-1.0 4.0 0.5" rpy="0 0 0"/>
   </joint>
-  <joint name="base_to_front_left_wheel" type="continuous">
+<!--############## selber gemacht #######-->
+<joint name="base_to_front_right_wheel" type="continuous">
+	<parent link="base_link"/>
+	<child link="front_right_wheel"/>
+	<origin xyz="0.35 -0.275 -0.22" rpy="0 0 0"/>
+	<axis xyz="0 1 0"/>
+</joint>
+<joint name="base_to_front_left_wheel" type="continuous">
+	<parent link="base_link"/>
+	<child link="front_left_wheel"/>
+	<origin xyz="0.35 0.275 -0.22" rpy="0 0 0"/>
+	<axis xyz="0 1 0"/>
+</joint>
+<joint name="base_to_rear_right_wheel" type="continuous">
+	<parent link="base_link"/>
+	<child link="rear_right_wheel"/>
+	<origin xyz="-0.35 -0.275 -0.22" rpy="0 0 0"/>
+	<axis xyz="0 1 0"/>
+</joint>
+<joint name="base_to_rear_left_wheel" type="continuous">
+	<parent link="base_link"/>
+	<child link="rear_left_wheel"/>
+	<origin xyz="-0.35 0.275 -0.22" rpy="0 0 0"/>
+	<axis xyz="0 1 0"/>
+</joint>
+<!--#####################-->
+  <joint name="base_to_camera" type="fixed">
     <parent link="base_link"/>
-    <child link="front_left_wheel"/>
-    <origin xyz="0.35 -0.275 -0.15"/>
-    <axis xyz="0 1 0"/>
-  </joint>
-  <joint name="base_to_front_right_wheel" type="continuous">
-    <parent link="base_link"/>
-    <child link="front_right_wheel"/>
-    <origin xyz="0.35 0.275 -0.15"/>
-    <axis xyz="0 1 0"/>
-  </joint>
-  <joint name="base_to_rear_right_wheel" type="continuous">
-    <parent link="base_link"/>
-    <child link="rear_right_wheel"/>
-    <origin xyz="-0.35 0.275 -0.15"/>
-    <axis xyz="0 1 0"/>
-  </joint>
-  <joint name="base_to_rear_left_wheel" type="continuous">
-    <parent link="base_link"/>
-    <child link="rear_left_wheel"/>
-    <origin xyz="-0.35 -0.275 -0.15"/>
-    <axis xyz="0 1 0"/>
+    <child link="camera_link"/>
+    <origin xyz="0.55 0 0"/>
   </joint>
   <joint name="base_to_lidar" type="fixed">
     <parent link="base_link"/>
     <child link="lidar"/>
-    <origin xyz="0 0 0.175"/>
+    <origin xyz="-0.5 0 0.3"/>
   </joint>
 <!--############################################ Aufruf von Makros ###################################-->
@@ -202,4 +233,5 @@
  <xacro:skid_steer_drive_controller/>
  <xacro:gazebo_ros_controller/>
+ <xacro:gazebo_camera/>
  <xacro:gazebo_lidar/>
 </robot>
